File: pcb/tomu-fpga/tomu-fpga.sch (KiCad schematic (older format))
At the start: 28 parts, among them P1 Captouch Pads, U1 LDO-SOT23-3.3V, U2 LDO-SOT23-2.5V, U3 LDO-SOT23-1.2V, U4 ICE40UP5K-SG48ITR, U5 Oscillator, U6 USB-B, U7 SPI-ROM, U8 RGB-LED

Commit message: pcb: sch: initial beta draft
This is the first feature-complete version of the schematic.

Signed-off-by: Sean Cross <sean@xobs.io>
Parts:
- added J1: Debug Header, symbol Connector_Generic:Conn_01x06
- added R1: 10k, 1/16W, 0201, symbol Device:R_Small
- added SW1: USER1, symbol Switch:SW_Push
- added SW2: USER2, symbol Switch:SW_Push
- added TP1, TP2, TP3, TP5: Testpoint, symbol tomu-fpga:Testpoint
- renumbered C3 to C1, C12 to C11, C4 to C12, C5 to C13, C1 to C2, C2 to C3, C13 to C4, C8 to C5, C11 to C8, R1 to R2, R2 to R3, R3 to R4, R4 to R5, TP1 to TP4, TP2 to TP6, U3 to U1, U1 to U2, U2 to U3, U7 to U4, U4 to U5, U5 to U6, U6 to U7
Connections:
- wire segments 158 -> 200
- no-connect marks 22 -> 14
Other:
- note added: "Developer I/O"
- note added: "Oscillator and Captouch"
- note added: "Power sequencing:\n1) 1.2V (VCC/VCCPLL)\n2) 3.3V (SPI_VCCIO1)\n3) 2.5V (VPP_2V5)\nSubsequent rails activate\nafter previous rail goes >0.5V"
- note added: "User I/O"
- note removed: "USB and LED"

Commit message: pcb: sch: finish evt1 schematic
This should be a feature-complete schematic.  Now to start on PCB
layout.

Signed-off-by: Sean Cross <sean@xobs.io>
Parts:
- removed C5, C6, C7: 0201, 1uF, 10V, X5R, 20%, symbol Device:C_Small
- added C11, C14, C17, C18, C23: 0201, 100nF, 10V, X5R, 20%, symbol Device:C_Small
- added C12, C15, C19, C8: 0201, 1uF, 10V, X5R, 20%, symbol Device:C_Small
- added C13, C16, C22, C9: 0201, 10nF, 10V, X5R, 20%, symbol Device:C_Small
- added R2: 10k, 1/16W, 0201, symbol Device:R_Small
- added R3, R4: 10k, 1/16W, 0201 (DNP), symbol Device:R_Small
- added R5: 1.5k, 1/16W, 0201, symbol Device:R_Small
- C5: renamed from C8; value 0201, 1uF, 6V, X5R, 20% -> 0201, 1uF, 10V, X5R, 20%
- C6: renamed from C9; value 0201, 1uF, 6V, X5R, 20% -> 0201, 1uF, 10V, X5R, 20%
- C7: renamed from C10; value 0201, 1uF, 6V, X5R, 20% -> 0201, 1uF, 10V, X5R, 20%
- R1: value 10k, 1/16W, 0201 -> 10k, 1/16W, 0201 (DNP)
- renumbered C11 to C10, C12 to C20, C13 to C21, R3 to R6, R4 to R7, R5 to R8, R2 to R9
Connections:
- net labels added: USBN_PU_CTRL
- wire segments 200 -> 250
- no-connect marks 14 -> 13
Other:
- note added: "Activate this PU to enable LS mode"
- note added: "VCCPLL Filter"
