File: hardware/tomu-fpga/tomu-fpga.sch (KiCad schematic (older format))
At the start: 50 parts, among them J1 Debug Header, P1 Captouch Pads, SW1 USER1, SW2 USER2, U1 LDO-SOT23-1.2V, U2 LDO-SOT23-3.3V, U3 LDO-SOT23-2.5V, U4 SPI-ROM, U5 ICE40UP5K-SG48ITR, U6 Oscillator, U7 USB-B, U8 RGB-LED

Commit message: hardware: pcb: add manufacturer and part numbers
Signed-off-by: Sean Cross <sean@xobs.io>
Parts:
- C1, C10, C11, C12, C13, C14, C15, C16, C17, C18, C19, C2, C21, C22, C23, C3, C4, C5, C6, C7, C8, C9: MPN (none) -> ANY; MYPN (none) -> ANY; Manufacturer (none) -> ANY
- C20: value 0201, 10uF, 6V, X5R, 20% -> 0201, 10uF, 10V, X5R, 20%; MPN (none) -> ANY; MYPN (none) -> ANY; Manufacturer (none) -> ANY
- J1, R1, R3, R4, TP1, TP2, TP3, TP4, TP5, TP6: MPN (none) -> DNP; MYPN (none) -> DNP; Manufacturer (none) -> DNP
- R2: value 10k, 1/16W, 0201 -> 10k, 1/16W, 0201 (DNP); MPN (none) -> DNP; MYPN (none) -> DNP; Manufacturer (none) -> DNP
- R5, R6: value 1.5k, 1/16W, 0201 -> 1.5k, 1/16W, 1%, 0201; MPN (none) -> ANY; MYPN (none) -> ANY; Manufacturer (none) -> ANY
- R7, R8: value 22ohm, 1/16W, 0201 -> 22ohm, 1/16W, 1%, 0201; MPN (none) -> ANY; MYPN (none) -> ANY; Manufacturer (none) -> ANY
- R9: value 100ohm, 1/16W, 0201 -> 100ohm, 1/16W, 1%, 0201; MPN (none) -> ANY; MYPN (none) -> ANY; Manufacturer (none) -> ANY
- U1: AMPN (none) -> MIC5504-1.2YMT; AManufacturer (none) -> Microchip; MPN (none) -> LP5907; Manufacturer (none) -> TI
- U2: AMPN (none) -> MIC5504-3.3YMT; AManufacturer (none) -> Microchip; MPN (none) -> LP5907; Manufacturer (none) -> TI
- U3: AMPN (none) -> MIC5504-2.5YMT; AManufacturer (none) -> Microchip; MPN (none) -> LP5907; Manufacturer (none) -> TI
- U5: MPN (none) -> ICE40UP5K-SG48ITR; Manufacturer (none) -> Lattice
- U6: value Oscillator -> MEMS Oscillator; MPN (none) -> DSC6001HI2A-048.0000T; Manufacturer (none) -> Digikey
- U8: MPN (none) -> UHD1110-FKA; Manufacturer (none) -> Cree
