File: hardware/pcb/tomu-fpga.sch (KiCad schematic (older format))
At the start: 50 parts, among them J1 Debug Header, P1 Captouch Pads, SW1 USER1, SW2 USER2, U1 LDO-SOT23-1.2V, U2 LDO-SOT23-3.3V, U3 LDO-SOT23-2.5V, U4 SPI-ROM, U5 ICE40UP5K-SG48ITR, U6 MEMS Oscillator, U7 USB-B, U8 RGB-LED

Commit message: pcb: sch: renumber schematic
Renumber the schematic again, as things have shifted around a bit.

Signed-off-by: Sean Cross <sean@xobs.io>
Parts:
- renumbered C9 to C10, C10 to C9
Changed lines of the file:
@@
 	4500 1750 4050 1750
 $Comp
-L Device:C_Small C10
+L Device:C_Small C9
 U 1 1 5BDE79EE
 P 5050 2100
-F 0 "C10" H 5100 2200 50  0000 L CNN
+F 0 "C9" H 5100 2200 50  0000 L CNN
 F 1 "0201, 100nF, 10V, X5R, 20%" H 4450 2300 50  0000 L CNN
 F 2 "" H 5050 2100 50  0001 C CNN
@@
 	4900 2200 4850 2200
 $Comp
-L power:GND #PWR018
+L power:GND #PWR017
 U 1 1 5BDEBDAC
 P 4900 2350
-F 0 "#PWR018" H 4900 2100 50  0001 C CNN
+F 0 "#PWR017" H 4900 2100 50  0001 C CNN
 F 1 "GND" H 4905 2177 50  0000 C CNN
 F 2 "" H 4900 2350 50  0001 C CNN
@@
 P 8800 4400
 F 0 "R9" H 8700 4300 50  0000 C CNN
-F 1 "100ohm, 1/16W, 1%, 0201" H 8300 4400 50  0000 C CNN
+F 1 "100ohm, 1/16W, 1%, 0201" H 9350 4300 50  0000 C CNN
 F 2 "" H 8800 4400 50  0001 C CNN
 F 3 "" H 8800 4400 50  0001 C CNN
@@
 $EndComp
 $Comp
-L power:GND #PWR020
+L power:GND #PWR019
 U 1 1 5C3C4455
 P 5400 7200
-F 0 "#PWR020" H 5400 6950 50  0001 C CNN
+F 0 "#PWR019" H 5400 6950 50  0001 C CNN
 F 1 "GND" H 5405 7027 50  0000 C CNN
 F 2 "" H 5400 7200 50  0001 C CNN
@@
 	2000 1300 2350 1300
 $Comp
-L power:+3V3 #PWR019
+L power:+3V3 #PWR018
 U 1 1 5C488914
 P 5400 6700
-F 0 "#PWR019" H 5400 6550 50  0001 C CNN
+F 0 "#PWR018" H 5400 6550 50  0001 C CNN
 F 1 "+3V3" H 5415 6873 50  0000 C CNN
 F 2 "" H 5400 6700 50  0001 C CNN
@@
 	5950 1650 5700 1650
 $Comp
-L power:GND #PWR021
+L power:GND #PWR020
 U 1 1 5C78A49F
 P 5700 1750
-F 0 "#PWR021" H 5700 1500 50  0001 C CNN
+F 0 "#PWR020" H 5700 1500 50  0001 C CNN
 F 1 "GND" H 5705 1577 50  0000 C CNN
 F 2 "" H 5700 1750 50  0001 C CNN
@@
 $EndComp
 $Comp
-L Device:C_Small C9
+L Device:C_Small C10
 U 1 1 5C8902B0
 P 5050 4450
-F 0 "C9" H 4900 4500 50  0000 L CNN
+F 0 "C10" H 4900 4500 50  0000 L CNN
 F 1 "0201, 10nF, 10V, X5R, 20%" H 4300 4600 50  0000 L CNN
 F 2 "" H 5050 4450 50  0001 C CNN
@@
 Connection ~ 5050 4550
 $Comp
-L power:GND #PWR017
+L power:GND #PWR021
 U 1 1 5C8902C6
 P 5750 4800
-F 0 "#PWR017" H 5750 4550 50  0001 C CNN
+F 0 "#PWR021" H 5750 4550 50  0001 C CNN
 F 1 "GND" H 5755 4627 50  0000 C CNN
 F 2 "" H 5750 4800 50  0001 C CNN

Commit message: hardware: sch: specify spinor part
SPINOR parts are largely interchangeable.  Pick one.

Signed-off-by: Sean Cross <sean@xobs.io>
Parts:
- U4: MPN (none) -> W25Q128JVSIM; Manufacturer (none) -> Winbond Electronics
Changed lines of the file:
@@
 F 1 "SPI-ROM" H 2100 6850 50  0000 C CNN
 F 2 "" H 2250 7000 50  0001 C CNN
-F 3 "" H 2250 7000 50  0001 C CNN
+F 3 "http://www.winbond.com/resource-files/w25q128jv_dtr%20revc%2003272018%20plus.pdf" H 2250 7000 50  0001 C CNN
+F 4 "W25Q128JVSIM " H 2450 7000 50  0001 C CNN "MPN"
+F 5 "Winbond Electronics" H 2450 7000 50  0001 C CNN "Manufacturer"
 	1    2450 7000
 	1    0    0    -1

Commit message: hardware: sch: add crystal, VCCPLL regulator
Add a crystal, so we can test to make sure it works.

Also add a second regulator dedicated to VCCPLL in an effort to
cost-down the capacitor and large components that shouldn't be
necessary.

Signed-off-by: Sean Cross <sean@xobs.io>
Parts:
- added C16, C19, C26: 0201, 1uF, 10V, X5R, 20%, symbol Device:C_Small
- added C28: 0201, 10nF, 10V, X5R, 20%, symbol Device:C_Small
- added C8: 0201, 100nF, 10V, X5R, 20%, symbol Device:C_Small
- added R2, R5: 0ohm (DNP), symbol Device:R_Small
- added U7: Crystal Oscillator, symbol tomu-fpga:Oscillator
- added U9: LDO-SOT23-1.2V, symbol tomu-fpga:LDO-SOT23
- C23: renamed from C20; value 0201, 10uF, 10V, X5R, 20% -> 0201, 10uF, 10V, X5R, 20% (DNP); MPN ANY -> DNP; MYPN ANY -> DNP; Manufacturer ANY -> DNP
- C24: renamed from C21; value 0201, 100nF, 10V, X5R, 20% -> 0201, 100nF, 10V, X5R, 20% (DNP); MPN ANY -> DNP; MYPN ANY -> DNP; Manufacturer ANY -> DNP
- R11: renamed from R9; value 100ohm, 1/16W, 1%, 0201 -> 100ohm, 1/16W, 1%, 0201 (DNP); MPN ANY -> DNP; MYPN ANY -> DNP; Manufacturer ANY -> DNP
- SW1: renamed from P1; DPN (none) -> CKN9104CT-ND
- SW2: renamed from SW1; MPN (none) -> PTS525SM15SMTR2 LFS; MYPN (none) -> SW-PB-5X5-1.6; Manufacturer (none) -> C&K
- SW3: renamed from SW2; DPN (none) -> CKN9104CT-ND; MPN (none) -> PTS525SM15SMTR2 LFS; MYPN (none) -> SW-PB-5X5-1.6; Manufacturer (none) -> C&K
- U1: DPN (none) -> 296-39062-1-ND; MPN LP5907 -> LP5907MFX-1.2/NOPB
- U2: DPN (none) -> 296-38557-1-ND; MPN LP5907 -> LP5907MFX-3.3/NOPB
- U3: DPN (none) -> 296-40356-1-ND; MPN LP5907 -> LP5907MFX-2.5/NOPB
- U4: DPN (none) -> W25Q128JVSIMCT-ND; MPN W25Q128JVSIM -> W25Q128JVSIM
- U5: value ICE40UP5K-SG48ITR -> ICE40UP5K-SG48I; symbol FPGA_Lattice:ICE40UP5K-SG48ITR -> Tomu_FPGA:ICE40UP5K-SG48ITR; DPN (none) -> 220-2212-1-ND; MPN (none) -> ICE40UP5K-SG48I; Manufacturer (none) -> Lattice
- U5: value ICE40UP5K-SG48ITR -> ICE40UP5K-SG48I; symbol FPGA_Lattice:ICE40UP5K-SG48ITR -> Tomu_FPGA:ICE40UP5K-SG48ITR; DPN (none) -> 220-2212-1-ND; MPN ICE40UP5K-SG48ITR -> ICE40UP5K-SG48I
- U6: DPN (none) -> DSC6001HI2A-048.0000T-ND; Manufacturer Digikey -> Microchip
- renumbered C9 to C10, C10 to C11, C11 to C12, C12 to C13, C13 to C14, C14 to C15, C15 to C17, C16 to C18, C17 to C20, C18 to C21, C19 to C22, C22 to C25, C23 to C27, C8 to C9, R8 to R10, R2 to R3, R3 to R4, R4 to R6, R5 to R7, R6 to R8, R7 to R9, U8 to U10, U7 to U8
Connections:
- wire segments 250 -> 291
Other:
- note added: "Main Power Rails"
- note added: "Note: Only populate regulator or filter circuit\nDo not populate both!"
- note added: "VCCPLL Regulator"
- note removed: "Power"
- moved on the sheet: C17, C18, C20, C21, SW1

Commit message: hardware: sch: populate SPI, /RESET pullups
It turns out these resistors are important.

Signed-off-by: Sean Cross <sean@xobs.io>
Parts:
- R1, R3: value 10k, 1/16W, 0201 (DNP) -> 10k, 1/16W, 0201; MPN DNP -> ANY; MYPN DNP -> ANY; Manufacturer DNP -> ANY
Changed lines of the file:
@@
 P 3550 5000
 F 0 "R1" H 3450 5050 50  0000 C CNN
-F 1 "10k, 1/16W, 0201 (DNP)" H 3800 4900 50  0000 C CNN
+F 1 "10k, 1/16W, 0201" H 3700 4900 50  0000 C CNN
 F 2 "" H 3550 5000 50  0001 C CNN
 F 3 "" H 3550 5000 50  0001 C CNN
-F 4 "DNP" H 3550 5000 50  0001 C CNN "MPN"
-F 5 "DNP" H 3550 5000 50  0001 C CNN "Manufacturer"
-F 6 "DNP" H 0   0   50  0001 C CNN "MYPN"
+F 4 "ANY" H 3550 5000 50  0001 C CNN "MPN"
+F 5 "ANY" H 3550 5000 50  0001 C CNN "Manufacturer"
+F 6 "ANY" H 0   0   50  0001 C CNN "MYPN"
 	1    3550 5000
 	-1   0    0    1
@@
 P 5000 7150
 F 0 "R4" V 4900 7150 50  0000 C CNN
-F 1 "10k, 1/16W, 0201 (DNP)" V 4800 7550 50  0000 C CNN
+F 1 "10k, 1/16W, 0201 (DNP)" V 4800 7450 50  0000 C CNN
 F 2 "" H 5000 7150 50  0001 C CNN
 F 3 "" H 5000 7150 50  0001 C CNN
@@
 P 5000 6850
 F 0 "R3" V 4900 6850 50  0000 C CNN
-F 1 "10k, 1/16W, 0201 (DNP)" V 5100 6850 50  0000 C CNN
+F 1 "10k, 1/16W, 0201" V 5100 6850 50  0000 C CNN
 F 2 "" H 5000 6850 50  0001 C CNN
 F 3 "" H 5000 6850 50  0001 C CNN
-F 4 "DNP" H 0   0   50  0001 C CNN "MPN"
-F 5 "DNP" H 0   0   50  0001 C CNN "MYPN"
-F 6 "DNP" H 0   0   50  0001 C CNN "Manufacturer"
+F 4 "ANY" H 0   0   50  0001 C CNN "MPN"
+F 5 "ANY" H 0   0   50  0001 C CNN "MYPN"
+F 6 "ANY" H 0   0   50  0001 C CNN "Manufacturer"
 	1    5000 6850
 	0    -1   -1   0

Commit message: hardware: pcb: add SPI debug header
This will be used to program SPI during board bringup.

Signed-off-by: Sean Cross <sean@xobs.io>
Parts:
- removed U5: ICE40UP5K-SG48I, Package_DFN_QFN:QFN-48-1EP_7x7mm_P0.5mm_EP5.6x5.6mm, symbol Tomu_FPGA:ICE40UP5K-SG48ITR
- added J1: SPI Header, Pin_Headers:Pin_Header_Angled_1x06_Pitch2.54mm, symbol Connector_Generic:Conn_01x10
- added U5: ICE40UP5K-SG48I, Package_DFN_QFN:QFN-48-1EP_7x7mm_P0.5mm_EP5.6x5.6mm, symbol tomu-fpga:ICE40UP5K-SG48ITR
- J2: renamed from J1; footprint (none) -> Pin_Headers:Pin_Header_Angled_1x10_Pitch2.54mm
Connections:
- net labels added: CDONE, CRESET
- wire segments 291 -> 302

Commit message: hardware: sch: use raspberry pi header, rework signaling
Rework the signaling to send everything to a Raspberry Pi header.

Signed-off-by: Sean Cross <sean@xobs.io>
Parts:
- removed J1: SPI Header, Pin_Headers:Pin_Header_Angled_1x06_Pitch2.54mm, symbol Connector_Generic:Conn_01x10
- removed J2: Debug Header, Pin_Headers:Pin_Header_Angled_1x10_Pitch2.54mm, symbol Connector_Generic:Conn_01x06
- removed TP1, TP2, TP3, TP5: Testpoint, symbol tomu-fpga:Testpoint
- removed U4: SPI-ROM, symbol tomu-fpga:SPI-ROM
- added D1: Power LED, symbol Device:LED
- added J1: Raspberry_Pi_2_3, symbol Connector:Raspberry_Pi_2_3
- added R2: 0805, 1.5k, 1/16W, 1%, symbol Device:R_Small
- added SW1: RESET, symbol Switch:SW_Push
- added U4: SPI Flash, symbol tomu-fpga:SPI-Flash
- C1, C13, C16, C17, C19, C2, C3: value 0201, 1uF, 10V, X5R, 20% -> 0805, 1uF, 10V, X5R, 20%
- C10: renamed from C7; value 0201, 1uF, 10V, X5R, 20% -> 0805, 1uF, 10V, X5R, 20%
- C11: renamed from C8; value 0201, 100nF, 10V, X5R, 20% -> 0805, 100nF, 10V, X5R, 20%
- C12: renamed from C10; value 0201, 100nF, 10V, X5R, 20% -> 0805, 100nF, 10V, X5R, 20%
- C14, C18: value 0201, 10nF, 10V, X5R, 20% -> 0805, 10nF, 10V, X5R, 20%
- C15, C20, C21, C4: value 0201, 100nF, 10V, X5R, 20% -> 0805, 100nF, 10V, X5R, 20%
- C22: renamed from C23; value 0201, 10uF, 10V, X5R, 20% (DNP) -> 0805, 10uF, 10V, X5R, 20% (DNP)
- C23: renamed from C24; value 0201, 100nF, 10V, X5R, 20% (DNP) -> 0805, 100nF, 10V, X5R, 20% (DNP)
- C24: renamed from C22; value 0201, 1uF, 10V, X5R, 20% -> 0805, 1uF, 10V, X5R, 20%
- C25: renamed from C26; value 0201, 1uF, 10V, X5R, 20% -> 0805, 1uF, 10V, X5R, 20%
- C26: renamed from C25; value 0201, 10nF, 10V, X5R, 20% -> 0805, 10nF, 10V, X5R, 20%
- C27: renamed from C28; value 0201, 10nF, 10V, X5R, 20% -> 0805, 10nF, 10V, X5R, 20%
- C28: renamed from C27; value 0201, 100nF, 10V, X5R, 20% -> 0805, 100nF, 10V, X5R, 20%
- C5: renamed from C9; value 0201, 1uF, 10V, X5R, 20% -> 0805, 1uF, 10V, X5R, 20%
- C6: renamed from C11; value 0201, 10nF, 10V, X5R, 20% -> 0805, 10nF, 10V, X5R, 20%
- C7: renamed from C12; value 0201, 100nF, 10V, X5R, 20% -> 0805, 100nF, 10V, X5R, 20%
- C8: renamed from C5; value 0201, 1uF, 10V, X5R, 20% -> 0805, 1uF, 10V, X5R, 20%
- C9: renamed from C6; value 0201, 1uF, 10V, X5R, 20% -> 0805, 1uF, 10V, X5R, 20%
- R1: value 10k, 1/16W, 0201 -> 0805, 10k, 1/16W
- R10: renamed from R11; value 100ohm, 1/16W, 1%, 0201 (DNP) -> 0805, 100ohm, 1/16W, 1% (DNP)
- R11: renamed from R9; value 22ohm, 1/16W, 1%, 0201 -> 0805, 22ohm, 1/16W, 1%
- R12: renamed from R10; value 22ohm, 1/16W, 1%, 0201 -> 0805, 22ohm, 1/16W, 1%
- R3: renamed from R4; value 10k, 1/16W, 0201 (DNP) -> 0805, 10k, 1/16W (DNP)
- R4: renamed from R6; value 10k, 1/16W, 0201 (DNP) -> 0805, 10k, 1/16W (DNP)
- R5: renamed from R3; value 10k, 1/16W, 0201 -> 0805, 10k, 1/16W
- R6: renamed from R2; value 0ohm (DNP) -> 0805, 0ohm (DNP)
- R7: renamed from R5; value 0ohm (DNP) -> 0805, 0ohm (DNP)
- R8: renamed from R7; value 1.5k, 1/16W, 1%, 0201 -> 0805, 1.5k, 1/16W, 1%
- R9: renamed from R8; value 1.5k, 1/16W, 1%, 0201 -> 0805, 1.5k, 1/16W, 1%
- renumbered SW1 to SW2, SW2 to SW3, SW3 to SW4, TP4 to TP1, TP6 to TP2, U9 to U8, U8 to U9
Connections:
- net labels added: DBG_1, DBG_2, DBG_3, DBG_4, DBG_5, DBG_6, UART_RX, UART_TX
- wire segments 302 -> 315
- no-connect marks 13 -> 25
Other:
- note added: "Boot and Reset"
- note added: "FPGA Power Input"
- note added: "PCB Power Regulation"
- note added: "Raspberry Pi "Hat"\nUsed for firmware development"
- note added: "To program SPI flash, put FPGA in RESET\nTo program FPGA, keep SPI_IO3 LOW"
- note removed: "Developer I/O"
- note removed: "Main Power Rails"
- note removed: "Power Regulation"
- moved on the sheet: C1, C10, C11, C12, C13, C14, C15, C16, C17, C18, C19, C2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

Commit message: pcb: hook up more debug wires
We have spare pins, so run more debug wires.

Many of these will probably get cut when doing the PCB layout.

Signed-off-by: Sean Cross <sean@xobs.io>
Connections:
- net labels added: DBG_10, DBG_11, DBG_12, DBG_13, DBG_14, DBG_15, DBG_16, DBG_17, DBG_18, DBG_7, DBG_8, DBG_9
- wire segments 315 -> 337
- no-connect marks 25 -> 3
Other:
- moved on the sheet: R9
Changed lines of the file:
@@
 L power:GND #PWR035
 U 1 1 5BD8C8EF
-P 8850 2200
-F 0 "#PWR035" H 8850 1950 50  0001 C CNN
-F 1 "GND" H 8855 2027 50  0000 C CNN
-F 2 "" H 8850 2200 50  0001 C CNN
-F 3 "" H 8850 2200 50  0001 C CNN
-	1    8850 2200
+P 8850 2050
+F 0 "#PWR035" H 8850 1800 50  0001 C CNN
+F 1 "GND" H 8855 1877 50  0000 C CNN
+F 2 "" H 8850 2050 50  0001 C CNN
+F 3 "" H 8850 2050 50  0001 C CNN
+	1    8850 2050
 	1    0    0    -1
 $EndComp
@@
 P 9400 1900
 F 0 "R12" V 9500 1900 50  0000 C CNN
-F 1 "0805, 22ohm, 1/16W, 1%" V 9550 1950 50  0000 C CNN
+F 1 "0805, 22ohm, 1/16W, 1%" V 9550 2000 50  0000 C CNN
 F 2 "" H 9400 1900 50  0001 C CNN
 F 3 "" H 9400 1900 50  0001 C CNN
@@
 Wire Wire Line
 	9500 1800 10000 1800
-Wire Wire Line
-	8700 1900 9000 1900
 Text Label 9600 1900 0    50   ~ 0
 ICE_USBP
@@
 Wire Wire Line
 	8850 1700 8700 1700
-Wire Wire Line
-	10000 2100 9850 2100
-Wire Wire Line
-	9850 2100 9850 2300
 $Comp
 L Device:R_Small R9
 U 1 1 5BDC6632
-P 9150 2300
-F 0 "R9" V 9250 2250 50  0000 C CNN
-F 1 "0805, 1.5k, 1/16W, 1%" V 9350 2550 50  0000 C CNN
-F 2 "" H 9150 2300 50  0001 C CNN
-F 3 "" H 9150 2300 50  0001 C CNN
-F 4 "ANY" H 650 100 50  0001 C CNN "MPN"
-F 5 "ANY" H 650 100 50  0001 C CNN "MYPN"
-F 6 "ANY" H 650 100 50  0001 C CNN "Manufacturer"
-	1    9150 2300
+P 9150 2350
+F 0 "R9" V 9050 2300 50  0000 C CNN
+F 1 "0805, 1.5k, 1/16W, 1%" V 9250 2350 50  0000 C CNN
+F 2 "" H 9150 2350 50  0001 C CNN
+F 3 "" H 9150 2350 50  0001 C CNN
+F 4 "ANY" H 650 150 50  0001 C CNN "MPN"
+F 5 "ANY" H 650 150 50  0001 C CNN "MYPN"
+F 6 "ANY" H 650 150 50  0001 C CNN "Manufacturer"
+	1    9150 2350
 	0    1    1    0
 $EndComp
-Wire Wire Line
-	9000 2300 9000 1900
-Wire Wire Line
-	9000 2300 9050 2300
-Connection ~ 9000 1900
-Wire Wire Line
-	9000 1900 9300 1900
-Wire Wire Line
-	9850 2300 9250 2300
-Text Label 9250 2300 0    50   ~ 0
+Text Label 9600 2200 2    50   ~ 0
 USBP_PU_CTRL
 Wire Wire Line
@@
 	0    1    1    0
 $EndComp
-NoConn ~ 10000 2900
-NoConn ~ 10000 2800
-NoConn ~ 10000 2500
-NoConn ~ 10000 2400
-NoConn ~ 10000 2300
-NoConn ~ 10000 2200
-NoConn ~ 5850 2150
 Wire Wire Line
 	8850 1550 8850 1700
@@
 	3150 4950 3150 4850
 Wire Wire Line
-	8850 2000 8850 2200
+	8850 2000 8850 2050
 Wire Notes Line
 	4100 600  7150 600
@@
 $EndComp
 $Comp
-L tomu-fpga:ICE40UP5K-SG48ITR U5
-U 1 1 5C1225F9
-P 10400 2400
-F 0 "U5" H 10100 1250 50  0000 L CNN
-F 1 "ICE40UP5K-SG48I" H 10100 1150 50  0000 L CNN
-F 2 "Package_DFN_QFN:QFN-48-1EP_7x7mm_P0.5mm_EP5.6x5.6mm" H 10400 1050 50  0001 C CNN
-F 3 "http://www.latticesemi.com/Products/FPGAandCPLD/iCE40Ultra" H 10000 3400 50  0001 C CNN
-F 4 "ICE40UP5K-SG48I" H 650 100 50  0001 C CNN "MPN"
-F 5 "220-2212-1-ND" H 650 100 50  0001 C CNN "DPN"
-F 6 "Lattice" H 650 100 50  0001 C CNN "Manufacturer"
-	1    10400 2400
-	1    0    0    -1
-$EndComp
-$Comp
-L Connector:Raspberry_Pi_2_3 J1
-U 1 1 5C14D2BF
-P 5600 5400
-F 0 "J1" H 4950 6650 50  0000 C CNN
-F 1 "Raspberry_Pi_2_3" H 6150 6650 50  0000 C CNN
-F 2 "" H 5600 5400 50  0001 C CNN
-F 3 "https://www.raspberrypi.org/documentation/hardware/raspberrypi/schematics/rpi_SCH_3bplus_1p0_reduced.pdf" H 5600 5400 50  0001 C CNN
-	1    5600 5400
-	1    0    0    -1
-$EndComp
-$Comp
 L tomu-fpga:SPI-Flash U4
 U 1 1 5C1645BF
@@
 Wire Wire Line
 	1700 4600 1900 4600
-NoConn ~ 4800 4800
-NoConn ~ 4800 5200
-NoConn ~ 4800 5300
-NoConn ~ 4800 5400
-NoConn ~ 4800 6000
-NoConn ~ 6400 6100
-NoConn ~ 6400 6200
-NoConn ~ 6400 4500
-NoConn ~ 6400 4600
-NoConn ~ 6400 5200
-NoConn ~ 6400 5300
-NoConn ~ 6400 5500
-NoConn ~ 2650 5850
-NoConn ~ 2650 5950
-NoConn ~ 2650 6050
-NoConn ~ 2650 6350
 Wire Wire Line
 	4800 5700 4450 5700
@@
 	3400 3600 2500 3600
 Connection ~ 2500 3600
+Wire Wire Line
+	6400 4500 6750 4500
+Wire Wire Line
+	6400 4600 6750 4600
+Wire Wire Line
+	6400 5200 6750 5200
+Wire Wire Line
+	6400 5300 6750 5300
+Text Label 6450 4500 0    50   ~ 0
+DBG_7
+Text Label 6450 4600 0    50   ~ 0
+DBG_8
+Text Label 6450 5200 0    50   ~ 0
+DBG_9
+Text Label 6450 5300 0    50   ~ 0
+DBG_10
+Wire Wire Line
+	6400 5500 6750 5500
+Text Label 6450 5500 0    50   ~ 0
+DBG_11
+Text Label 6450 6100 0    50   ~ 0
+DBG_12
+Text Label 6450 6200 0    50   ~ 0
+DBG_13
+Wire Wire Line
+	6400 6100 6750 6100
+Wire Wire Line
+	6400 6200 6750 6200
+$Comp
+L Connector:Raspberry_Pi_2_3 J1
+U 1 1 5C14D2BF
+P 5600 5400
+F 0 "J1" H 4950 6650 50  0000 C CNN
+F 1 "Raspberry_Pi_2_3" H 6150 6650 50  0000 C CNN
+F 2 "" H 5600 5400 50  0001 C CNN
+F 3 "https://www.raspberrypi.org/documentation/hardware/raspberrypi/schematics/rpi_SCH_3bplus_1p0_reduced.pdf" H 5600 5400 50  0001 C CNN
+	1    5600 5400
+	1    0    0    -1
+$EndComp
+Wire Wire Line
+	4800 6000 4450 6000
+Wire Wire Line
+	4800 5400 4450 5400
+Wire Wire Line
+	4800 5300 4450 5300
+Wire Wire Line
+	4800 5200 4450 5200
+Text Label 4450 6000 0    50   ~ 0
+DBG_14
+Text Label 4450 5400 0    50   ~ 0
+DBG_15
+Text Label 4450 5300 0    50   ~ 0
+DBG_16
+Text Label 4450 5200 0    50   ~ 0
+DBG_17
+Text Label 2300 6350 0    50   ~ 0
+DBG_7
+Text Label 2300 6050 0    50   ~ 0
+DBG_8
+Text Label 2300 5950 0    50   ~ 0
+DBG_9
+Text Label 2300 5850 0    50   ~ 0
+DBG_10
+Wire Wire Line
+	2300 5850 2650 5850
+Wire Wire Line
+	2650 5950 2300 5950
+Wire Wire Line
+	2300 6050 2650 6050
+Wire Wire Line
+	2650 6350 2300 6350
+Text Label 9650 2900 0    50   ~ 0
+DBG_11
+Text Label 9650 2800 0    50   ~ 0
+DBG_12
+Text Label 9650 2500 0    50   ~ 0
+DBG_13
+Text Label 9650 2400 0    50   ~ 0
+DBG_14
+Text Label 9650 2300 0    50   ~ 0
+DBG_15
+Text Label 9650 2200 0    50   ~ 0
+DBG_16
+Text Label 5550 2150 0    50   ~ 0
+DBG_17
+Text Label 7100 4500 0    50   ~ 0
+DBG_18
+$Comp
+L tomu-fpga:ICE40UP5K-SG48ITR U5
+U 1 1 5C1225F9
+P 10400 2400
+F 0 "U5" H 10100 1250 50  0000 L CNN
+F 1 "ICE40UP5K-SG48I" H 10100 1150 50  0000 L CNN
+F 2 "Package_DFN_QFN:QFN-48-1EP_7x7mm_P0.5mm_EP5.6x5.6mm" H 10400 1050 50  0001 C CNN
+F 3 "http://www.latticesemi.com/Products/FPGAandCPLD/iCE40Ultra" H 10000 3400 50  0001 C CNN
+F 4 "ICE40UP5K-SG48I" H 650 100 50  0001 C CNN "MPN"
+F 5 "220-2212-1-ND" H 650 100 50  0001 C CNN "DPN"
+F 6 "Lattice" H 650 100 50  0001 C CNN "Manufacturer"
+	1    10400 2400
+	1    0    0    -1
+$EndComp
+Wire Wire Line
+	8700 1900 9000 1900
+Connection ~ 9000 1900
+Wire Wire Line
+	9000 1900 9300 1900
+Wire Wire Line
+	9650 2500 10000 2500
+Wire Wire Line
+	10000 2400 9650 2400
+Wire Wire Line
+	9650 2300 10000 2300
+Wire Wire Line
+	10000 2200 9650 2200
+Wire Wire Line
+	5550 2150 5850 2150
+Wire Wire Line
+	9650 2800 10000 2800
+Wire Wire Line
+	10000 2900 9650 2900
+Wire Wire Line
+	9600 2100 9600 2350
+Wire Wire Line
+	9600 2100 10000 2100
+Wire Wire Line
+	9050 2350 9000 2350
+Wire Wire Line
+	9000 2350 9000 1900
+Wire Wire Line
+	9600 2350 9250 2350
+NoConn ~ 4800 4800
 $EndSCHEMATC

Commit message: hardware: add testpoints for SPI programming
This will become necessary when doing factory burning.

Signed-off-by: Sean Cross <sean@xobs.io>
Parts:
- added TP2, TP3, TP4, TP5, TP6, TP7: Testpoint, symbol tomu-fpga:Testpoint
- C1, C10, C11, C12, C13, C14, C15, C16, C17, C18, C19, C2, C20, C21, C22, C23, C24, C25, C26, C27, C28, C3, C4, C5, C6, C7, C8, C9: footprint (none) -> Capacitors_SMD:C_0805
- R1, R10, R11, R12, R2, R3, R4, R5, R6, R7, R8, R9: footprint (none) -> Resistors_SMD:R_0805
- renumbered TP2 to TP8
Connections:
- wire segments 337 -> 343
