File: hardware/pcb/tomu-fpga.sch (KiCad schematic (older format))
At the start: 64 parts, among them J1 Raspberry_Pi_2_3, SW1 RESET, SW2 Captouch Pads, SW3 USER1, SW4 USER2, U1 LDO-SOT23-1.2V, U10 RGB-LED, U2 LDO-SOT23-3.3V, U3 LDO-SOT23-2.5V, U4 SPI Flash, U5 ICE40UP5K-SG48I, U6 MEMS Oscillator, U7 Crystal Oscillator, U8 LDO-SOT23-1.2V, U9 USB-B

Commit message: hardware: sch: map remaining footprints
Add footprints for the remaining schematic components.

Signed-off-by: Sean Cross <sean@xobs.io>
Parts:
- D1: footprint (none) -> LEDs:LED_0805; DPN (none) -> 160-1415-1-ND; Description (none) -> LED RED CLEAR SMD; MPN (none) -> LTST-C170KRKT; Manufacturer (none) -> Lite-On Inc.
- J1: footprint (none) -> Pin_Headers:Pin_Header_Straight_1x20_Pitch2.54mm; Description (none) -> Connector for development
- SW1, SW4: footprint (none) -> tomu-fpga:SPST-NO-Button; Description (none) -> SWITCH TACTILE SPST-NO 0.02A 15V
- SW2: footprint (none) -> tomu-fpga:Touchpads; DPN CKN9104CT-ND -> (none); Description (none) -> PCB-etched captouch pads
- SW3: footprint (none) -> tomu-fpga:SPST-NO-Button; DPN (none) -> CKN9104CT-ND; Description (none) -> SWITCH TACTILE SPST-NO 0.02A 15V
- TP1, TP2, TP3, TP4, TP5, TP6, TP7, TP8: footprint (none) -> Measurement_Points:Measurement_Point_Round-SMD-Pad_Small
- U1, U8: footprint (none) -> TO_SOT_Packages_SMD:SOT-23-5_HandSoldering; Description (none) -> IC REG LINEAR 1.2V 250MA SOT23-5
- U10: footprint (none) -> tomu-fpga:LED-RGB-5DS-UHD1110-FKA; DPN (none) -> N/A
- U2: footprint (none) -> TO_SOT_Packages_SMD:SOT-23-5_HandSoldering; Description (none) -> IC REG LINEAR 3.3V 250MA SOT23-5
- U3: footprint (none) -> TO_SOT_Packages_SMD:SOT-23-5_HandSoldering; Description (none) -> IC REG LINEAR 2.5V 250MA SOT23-5
- U4: footprint (none) -> SMD_Packages:SOIC-8-N; Description (none) -> IC FLASH 128M SPI 133MHZ 8SOIC
- U5: Description (none) -> ICE40-ULTRAPLUS, 5280 LUTS, 1.2V
- U6: footprint (none) -> tomu-fpga:MEMS-20005625B; Description (none) -> MEMS OSC XO 48.0000MHZ CMOS SMD
- U7: footprint (none) -> tomu-fpga:XTAL-2520; Description (none) -> XTAL OSC XO 48.0000MHZ CMOS SMD
- U9: footprint (none) -> tomu-fpga:USB-B; Description (none) -> PCB-etched USB pads

Commit message: hardware: sch: use footprints from `tomu-fpga`
Use our local copy of footprints, which are guaranteed not to change
between Kicad versions.

Signed-off-by: Sean Cross <sean@xobs.io>
Parts:
- C1, C10, C11, C12, C13, C14, C15, C16, C17, C18, C19, C2, C20, C21, C22, C23, C24, C25, C26, C27, C28, C3, C4, C5, C6, C7, C8, C9: footprint Capacitors_SMD:C_0805 -> tomu-fpga:C_0805_2012Metric_Pad1.15x1.40mm_HandSolder
- D1: footprint LEDs:LED_0805 -> tomu-fpga:LED_0805_2012Metric_Pad1.15x1.40mm_HandSolder
- J1: footprint Pin_Headers:Pin_Header_Straight_1x20_Pitch2.54mm -> tomu-fpga:PinHeader_2x20_P2.54mm_Vertical
- R1, R10, R11, R12, R2, R3, R4, R5, R6, R7, R8, R9: footprint Resistors_SMD:R_0805 -> tomu-fpga:R_0805_2012Metric_Pad1.15x1.40mm_HandSolder
- TP1, TP2, TP3, TP4, TP5, TP6, TP7, TP8: footprint Measurement_Points:Measurement_Point_Round-SMD-Pad_Small -> tomu-fpga:TestPoint_Pad_D1.5mm
- U1, U2, U3, U8: footprint TO_SOT_Packages_SMD:SOT-23-5_HandSoldering -> tomu-fpga:SOT-23-5_HandSoldering
- U4: footprint SMD_Packages:SOIC-8-N -> tomu-fpga:SOIC-8
- U5: footprint Package_DFN_QFN:QFN-48-1EP_7x7mm_P0.5mm_EP5.6x5.6mm -> tomu-fpga:QFN-48-1EP_7x7mm_P0.5mm_EP5.6x5.6mm

Commit message: hardware: first fully-routed PCB
The PCB is terrible, and probably would have all sorts of issues.  Will
rip it up and try again tomorrow.

Signed-off-by: Sean Cross <sean@xobs.io>
Parts:
- removed C12: 0805, 100nF, 10V, X5R, 20%, tomu-fpga:C_0805_2012Metric_Pad1.15x1.40mm_HandSolder, symbol Device:C_Small
- removed TP1, TP2, TP3, TP4, TP5, TP6, TP7, TP8: Testpoint, tomu-fpga:TestPoint_Pad_D1.5mm, symbol tomu-fpga:Testpoint
- added R13: 0201, 0ohm (DNP), tomu-fpga:R_0201_0603Metric, symbol Device:R_Small
- R3: value 0805, 10k, 1/16W (DNP) -> 0201, 0ohm (DNP); footprint tomu-fpga:R_0805_2012Metric_Pad1.15x1.40mm_HandSolder -> tomu-fpga:R_0201_0603Metric
- R6, R7: value 0805, 0ohm (DNP) -> 0201, 0ohm (DNP); footprint tomu-fpga:R_0805_2012Metric_Pad1.15x1.40mm_HandSolder -> tomu-fpga:R_0201_0603Metric
- SW1, SW3, SW4: symbol Switch:SW_Push -> tomu-fpga:SW_Push
Connections:
- net labels added: LED_B, LED_G, LED_R, VCCPLL
- net labels removed: DBG_11, DBG_12, DBG_13, DBG_14, DBG_15, DBG_16, DBG_17, DBG_3, DBG_5, DBG_6
- wire segments 343 -> 339
- no-connect marks 3 -> 23
Other:
- moved on the sheet: R4, R5, R6, U6

Commit message: hardware: sch: add PMOD connector
Signed-off-by: Sean Cross <sean@xobs.io>
Parts:
- added J3: PMOD, Pin_Headers:Pin_Header_Straight_1x06_Pitch2.54mm, symbol Connector:Conn_01x06_Female
Connections:
- net labels added: PMOD_1, PMOD_2, PMOD_3, PMOD_4, PU_CTRL_USBN, PU_CTRL_USBP
- net labels removed: DBG_2, USBN_PU_CTRL, USBP_PU_CTRL
- wire segments 339 -> 353
- no-connect marks 23 -> 21
Other:
- moved on the sheet: R8, R9, SW2

Commit message: hardware: sch: provide APN for RGB LED
Provide an alternate part number for the RGB LED, since the current one
is hard to source.

Signed-off-by: Sean Cross <sean@xobs.io>
Parts:
- J3: footprint Pin_Headers:Pin_Header_Straight_1x06_Pitch2.54mm -> tomu-fpga:Pin_Header_Straight_1x06_Pitch2.54mm; symbol Connector:Conn_01x06_Female -> tomu-fpga:Conn_01x06_Female; DPN (none) -> DNP; MPN (none) -> DNP; Manufacturer (none) -> DNP
- U10: AManufacturer (none) -> Citizen; APN (none) -> CL-505S-X-SD-T
- U6: value MEMS Oscillator -> MEMS Oscillator (DNP)
Changed lines of the file:
@@
 U 1 1 5BD8B24F
 P 8300 1600
-F 0 "U9" H 8244 1485 50  0000 C CNN
-F 1 "USB-B" H 8244 1576 50  0000 C CNN
+F 0 "U9" H 8550 1600 50  0000 C CNN
+F 1 "USB-B" H 8150 1600 50  0000 C CNN
 F 2 "tomu-fpga:USB-B" H 8300 1600 50  0001 C CNN
 F 3 "" H 8300 1600 50  0001 C CNN
@@
 F 5 "Cree" H 9250 3450 50  0001 C CNN "Manufacturer"
 F 6 "N/A" H 0   0   50  0001 C CNN "DPN"
+F 7 "CL-505S-X-SD-T" H 9250 3450 50  0001 C CNN "APN"
+F 8 "Citizen" H 9250 3450 50  0001 C CNN "AManufacturer"
 	1    9250 3450
 	1    0    0    -1
@@
 P 4750 1600
 F 0 "U6" H 5050 1550 50  0000 C CNN
-F 1 "MEMS Oscillator" H 4650 1550 50  0000 C CNN
+F 1 "MEMS Oscillator (DNP)" H 4650 1550 50  0000 C CNN
 F 2 "tomu-fpga:MEMS-20005625B" H 4750 1600 50  0001 C CNN
 F 3 "http://ww1.microchip.com/downloads/en/DeviceDoc/20005625B.pdf" H 4750 1600 50  0001 C CNN
@@
 NoConn ~ 4800 5700
 $Comp
-L Connector:Conn_01x06_Female J3
+L tomu-fpga:Conn_01x06_Female J3
 U 1 1 5EC9746F
 P 7950 1150
-F 0 "J3" H 7900 750 50  0000 C CNN
-F 1 "PMOD" V 8000 1100 50  0000 C CNN
-F 2 "Pin_Headers:Pin_Header_Straight_1x06_Pitch2.54mm" H 7950 1150 50  0001 C CNN
+F 0 "J3" H 7950 750 50  0000 C CNN
+F 1 "PMOD" H 7900 1450 50  0000 C CNN
+F 2 "tomu-fpga:Pin_Header_Straight_1x06_Pitch2.54mm" H 7950 1150 50  0001 C CNN
 F 3 "~" H 7950 1150 50  0001 C CNN
+F 4 "DNP" H 7950 1150 50  0001 C CNN "MPN"
+F 5 "DNP" H 7950 1150 50  0001 C CNN "Manufacturer"
+F 6 "DNP" H 7950 1150 50  0001 C CNN "DPN"
 	1    7950 1150
 	-1   0    0    1

Commit message: hardware: fix USB footprint being mirrored
That could have been bad.

Signed-off-by: Sean Cross <sean@xobs.io>
Connections:
- wire segments 353 -> 355
Changed lines of the file:
@@
 	0    1    1    0
 $EndComp
-Text Label 9950 2800 2    50   ~ 0
+Text Label 9950 2700 2    50   ~ 0
 PU_CTRL_USBP
 $Comp
@@
 Wire Wire Line
 	9000 1800 9300 1800
-Text Label 9550 2700 1    50   ~ 0
+Text Label 9550 2600 1    50   ~ 0
 PU_CTRL_USBN
 Text Notes 8600 1200 0    50   ~ 0
@@
 Text Label 9650 2500 1    50   ~ 0
 ICE_USBP
-Text Label 9800 2500 1    50   ~ 0
+Text Label 9800 2450 1    50   ~ 0
 ICE_USBN
 Wire Wire Line
-	10000 2500 9800 2500
-Wire Wire Line
-	9350 2400 9350 2800
-Wire Wire Line
-	9350 2800 10000 2800
-Wire Wire Line
-	10000 2700 9550 2700
-Wire Wire Line
 	9550 1250 9550 2700
 Wire Wire Line
-	9800 2500 9800 1800
-Wire Wire Line
 	9500 1900 9650 1900
-Wire Wire Line
-	9650 2600 10000 2600
 Wire Wire Line
 	5750 2250 5750 1400
@@
 $EndComp
 Wire Wire Line
-	9650 1900 9650 2600
+	9650 1900 9650 2500
 Wire Wire Line
 	10000 1800 10000 1400
@@
 Wire Wire Line
 	8600 1250 8600 950
+Wire Wire Line
+	10000 2500 9800 2500
+Wire Wire Line
+	9800 2500 9650 2500
+Wire Wire Line
+	10000 2600 9800 2600
+Wire Wire Line
+	9800 1800 9800 2600
+Wire Wire Line
+	9350 2400 9350 2700
+Wire Wire Line
+	9550 2700 9550 2800
+Wire Wire Line
+	9550 2800 10000 2800
+Wire Wire Line
+	9350 2700 10000 2700
 $EndSCHEMATC

Commit message: hardware: sch: first draft of dvt1
This removes much of the support debugging stuff from evt1.  Still to
do:

- Assign footprints
- Figure out which PU resistor to include (if any)
- Figure out if we need to keep the USB buffering
- Remove extra decoupling caps

Signed-off-by: Sean Cross <sean@xobs.io>
Parts:
- removed C22: 0805, 10uF, 10V, X5R, 20% (DNP), tomu-fpga:C_0805_2012Metric_Pad1.15x1.40mm_HandSolder, symbol Device:C_Small
- removed C23: 0805, 100nF, 10V, X5R, 20% (DNP), tomu-fpga:C_0805_2012Metric_Pad1.15x1.40mm_HandSolder, symbol Device:C_Small
- removed D1: Power LED, tomu-fpga:LED_0805_2012Metric_Pad1.15x1.40mm_HandSolder, symbol Device:LED
- removed J1: Raspberry_Pi_2_3, tomu-fpga:PinHeader_2x20_P2.54mm_Vertical, symbol Connector:Raspberry_Pi_2_3
- removed J3: PMOD, tomu-fpga:Pin_Header_Straight_1x06_Pitch2.54mm, symbol tomu-fpga:Conn_01x06_Female
- removed R10: 0805, 100ohm, 1/16W, 1% (DNP), tomu-fpga:R_0805_2012Metric_Pad1.15x1.40mm_HandSolder, symbol Device:R_Small
- removed R2: 0805, 1.5k, 1/16W, 1%, tomu-fpga:R_0805_2012Metric_Pad1.15x1.40mm_HandSolder, symbol Device:R_Small
- removed R4: 0805, 10k, 1/16W (DNP), tomu-fpga:R_0805_2012Metric_Pad1.15x1.40mm_HandSolder, symbol Device:R_Small
- removed R6, R7: 0201, 0ohm (DNP), tomu-fpga:R_0201_0603Metric, symbol Device:R_Small
- removed SW1: RESET, tomu-fpga:SPST-NO-Button, symbol tomu-fpga:SW_Push
- removed SW3: USER1, tomu-fpga:SPST-NO-Button, symbol tomu-fpga:SW_Push
- removed SW4: USER2, tomu-fpga:SPST-NO-Button, symbol tomu-fpga:SW_Push
- removed U1, U8: LDO-SOT23-1.2V, tomu-fpga:SOT-23-5_HandSoldering, symbol tomu-fpga:LDO-SOT23
- removed U2: LDO-SOT23-3.3V, tomu-fpga:SOT-23-5_HandSoldering, symbol tomu-fpga:LDO-SOT23
- removed U3: LDO-SOT23-2.5V, tomu-fpga:SOT-23-5_HandSoldering, symbol tomu-fpga:LDO-SOT23
- removed U6: MEMS Oscillator (DNP), tomu-fpga:MEMS-20005625B, symbol tomu-fpga:Oscillator
- added TP1, TP10, TP11, TP12, TP2, TP3, TP4, TP5, TP6, TP7, TP8, TP9: Testpoint, symbol Tomu_FPGA:Testpoint
- added U1, U6: LDO-X2SON-1.2V, tomu-fpga:Texas_X2SON-4_1x1mm_P0.65mm, symbol Tomu_FPGA:LDO-X2SON
- added U2: LDO-X2SON-3.3V, tomu-fpga:Texas_X2SON-4_1x1mm_P0.65mm, symbol Tomu_FPGA:LDO-X2SON
- added U3: LDO-X2SON-2.5V, tomu-fpga:Texas_X2SON-4_1x1mm_P0.65mm, symbol Tomu_FPGA:LDO-X2SON
- C1, C10, C11, C13, C14, C15, C16, C17, C18, C19, C2, C20, C21, C24, C25, C26, C27, C28, C3, C4, C5, C6, C7, C8, C9: footprint tomu-fpga:C_0805_2012Metric_Pad1.15x1.40mm_HandSolder -> tomu-fpga:C_0201_0603Metric
- R1, R11, R12, R5, R8, R9: footprint tomu-fpga:R_0805_2012Metric_Pad1.15x1.40mm_HandSolder -> tomu-fpga:R_0201_0603Metric
Connections:
- net labels removed: DBG_1, DBG_10, DBG_4, DBG_7, DBG_8, DBG_9, PMOD_1, PMOD_2, PMOD_3, PMOD_4, UART_RX, UART_TX
- wire segments 355 -> 254
- no-connect marks 21 -> 22
Other:
- note removed: "Note: Only populate regulator or filter circuit\nDo not populate both!"
- note removed: "Raspberry Pi "Hat"\nUsed for firmware development"
- note removed: "VCCPLL Filter"
- note removed: "VCCPLL Regulator"
- moved on the sheet: SW2, U10

Commit message: hardware: sch: work-in-progress to go from QFN to WLCSP
Signed-off-by: Sean Cross <sean@xobs.io>
Parts:
- removed R13, R3: 0201, 0ohm (DNP), tomu-fpga:R_0201_0603Metric, symbol Device:R_Small
- removed R8: 0805, 1.5k, 1/16W, 1%, tomu-fpga:R_0201_0603Metric, symbol Device:R_Small
- C1, C10, C13, C16, C17, C19, C2, C24, C25, C3, C5, C8, C9: value 0805, 1uF, 10V, X5R, 20% -> 0201, 1uF, 10V, X5R, 20%
- C11, C15, C20, C21, C28, C4, C7: value 0805, 100nF, 10V, X5R, 20% -> 0201, 100nF, 10V, X5R, 20%
- C14, C18, C26, C27, C6: value 0805, 10nF, 10V, X5R, 20% -> 0201, 10nF, 10V, X5R, 20%
- R1, R5: value 0805, 10k, 1/16W -> 0201, 10k, 1/16W
- R11, R12: value 0805, 22ohm, 1/16W, 1% -> 0201, 22ohm, 1/16W, 1%
- R9: value 0805, 1.5k, 1/16W, 1% -> 0201, 1.5k, 1/16W, 1%
- TP1, TP10, TP11, TP12, TP2, TP3, TP4, TP5, TP6, TP7, TP8, TP9: symbol Tomu_FPGA:Testpoint -> tomu-fpga:Testpoint
- U1, U2, U3, U6: symbol Tomu_FPGA:LDO-X2SON -> tomu-fpga:LDO-X2SON
- U5: value ICE40UP5K-SG48I -> ICE40UP5K-UWG30; symbol tomu-fpga:ICE40UP5K-SG48ITR -> tomu-fpga:ICE40UP5K-UWG30; DPN 220-2212-1-ND -> ICE40UP5K-UWG30ITR-ND; MPN ICE40UP5K-SG48I -> ICE40UP5K-UWG30ITR
- U9: footprint tomu-fpga:USB-B -> tomu-fpga:USB-PCB
Connections:
- net labels added: TOUCH_1, TOUCH_2, TOUCH_3, TOUCH_4
- net labels removed: PU_CTRL_USBN
- wire segments 254 -> 242
- no-connect marks 22 -> 4
Other:
- note removed: "Activate this PU to enable LS mode"
- moved on the sheet: U10
