File: hardware/pcb/tomu-fpga.sch (KiCad schematic (older format))
At the start: 52 parts, among them SW2 Captouch Pads, U1 LDO-X2SON-1.2V, U10 RGB-LED, U2 LDO-X2SON-3.3V, U3 LDO-X2SON-2.5V, U4 SPI Flash, U5 ICE40UP5K-UWG30, U6 LDO-X2SON-1.2V, U7 Crystal Oscillator, U9 USB-B

Commit message: hardware: sch: complete schematic layout of DVT1
This is the first cut of a schematic layout of DVT1.

It includes all the decoupling caps still.  We'll need to see if they're
kept around.

Signed-off-by: Sean Cross <sean@xobs.io>
Parts:
- added XX1: Touchpad Mask Removal, tomu-fpga:soldermask-removal, symbol tomu-fpga:Touchpad-Note
- added XX2: Case, tomu-fpga:nothing, symbol tomu-fpga:Case
- added XX3: ESD Bag, tomu-fpga:nothing, symbol tomu-fpga:Case
- SW2: footprint tomu-fpga:Touchpads -> tomu-fpga:captouch-edge
- TP1, TP10, TP11, TP12, TP2, TP3, TP4, TP5, TP6, TP7, TP8, TP9: footprint (none) -> tomu-fpga:testpoint
- U4: footprint tomu-fpga:SOIC-8 -> tomu-fpga:USON8_2X3MM
- U5: footprint tomu-fpga:QFN-48-1EP_7x7mm_P0.5mm_EP5.6x5.6mm -> tomu-fpga:iCE40UP5K-UWG30
Connections:
- net labels removed: DBG_18
Other:
- note added: "Manufacturing Notes"
- note added: "Test Pads"

Commit message: hardware: schematic: rewire fpga as necessary for routing
FPGAs are great, because if there's an alternate method that's easier to
route -- go for it!  This modifies some of the connections to ease
routing constraints.

Signed-off-by: Sean Cross <sean@xobs.io>
Parts:
- U4: footprint tomu-fpga:USON8_2X3MM -> tomu-fpga:SON50P300X200X60-9N
Connections:
- net labels added: USB_N, USB_P
- wire segments 242 -> 236
- no-connect marks 4 -> 5
Changed lines of the file:
@@
 Text Label 9250 2400 0    50   ~ 0
 PU_CTRL_USBP
-Text Label 5550 2050 0    50   ~ 0
+Text Label 5400 2400 0    50   ~ 0
 OSC_IN
 Wire Wire Line
@@
 $EndComp
 Wire Wire Line
-	5850 2250 5400 2250
+	5850 2050 5250 2050
 $Comp
 L power:GND #PWR041
@@
 	4450 2750 4450 2600
 Connection ~ 4450 2600
-Wire Wire Line
-	5150 2400 5250 2400
-Wire Wire Line
-	5250 2050 5850 2050
 $Comp
 L Device:C_Small C11
@@
 F 0 "U4" H 1675 7815 50  0000 C CNN
 F 1 "SPI Flash" H 1675 7724 50  0000 C CNN
-F 2 "tomu-fpga:USON8_2X3MM" H 1450 7000 50  0001 C CNN
+F 2 "tomu-fpga:SON50P300X200X60-9N" H 1450 7000 50  0001 C CNN
 F 3 "http://www.winbond.com/resource-files/w25q128jv_dtr%20revc%2003272018%20plus.pdf" H 1450 7000 50  0001 C CNN
 F 4 "W25Q128JVSIMCT-ND" H -450 -1450 50  0001 C CNN "DPN"
@@
 LED_R
 Wire Wire Line
-	9850 2600 9700 2600
-Wire Wire Line
-	9700 2600 9700 2900
-Wire Wire Line
-	9700 2900 9400 2900
-Wire Wire Line
-	9850 2700 9600 2700
-Wire Wire Line
-	9600 2700 9600 2600
-Wire Wire Line
 	9500 2800 9500 2700
 Wire Wire Line
 	9500 2800 9850 2800
-Wire Wire Line
-	9400 2800 9400 2900
 Text Label 9550 1900 0    50   ~ 0
 ICE_USBP
@@
 $EndComp
 Wire Wire Line
-	9650 1900 9650 2300
-Wire Wire Line
-	9800 1800 9800 2200
-Wire Wire Line
-	5250 2050 5250 2400
+	9650 1900 9650 2200
 Wire Wire Line
 	4200 1600 4200 2600
-Wire Wire Line
-	5400 2250 5400 1500
-Wire Wire Line
-	5400 1500 5250 1500
-Wire Wire Line
-	5250 1500 5250 1400
 Text Notes 1150 7400 0    50   ~ 0
 To program SPI flash, put FPGA in RESET\nTo program FPGA, keep SPI_IO3 LOW
@@
 GND
 Text Label 5450 5900 0    50   ~ 0
-ICE_USBP
+USB_P
 Text Label 5450 5750 0    50   ~ 0
-ICE_USBN
+USB_N
 $Comp
 L tomu-fpga:Testpoint TP10
@@
 $EndComp
 NoConn ~ 2650 5950
-NoConn ~ 2650 6050
 NoConn ~ 1450 1200
 Wire Wire Line
@@
 Connection ~ 10850 5200
 Wire Wire Line
-	9850 2200 9800 2200
-Wire Wire Line
-	9850 2300 9650 2300
-Wire Wire Line
 	9850 2500 9800 2500
 Wire Wire Line
@@
 	9250 2400 9800 2400
 Wire Wire Line
-	8950 2800 9400 2800
+	8950 2800 9300 2800
 Wire Wire Line
 	8950 2700 9500 2700
 Wire Wire Line
-	8950 2600 9600 2600
-Wire Wire Line
 	8100 2400 8100 2600
 Wire Wire Line
@@
 Wire Wire Line
 	10450 1200 10850 1200
-Text Label 5500 2250 0    50   ~ 0
+Text Label 5250 1800 1    50   ~ 0
 TOUCH_4
 Text Label 5150 1800 1    50   ~ 0
@@
 Text Label 4950 1800 1    50   ~ 0
 TOUCH_1
-Text Label 2300 6350 0    50   ~ 0
-TOUCH_4
-Wire Wire Line
-	2650 6350 2300 6350
 NoConn ~ 9850 2400
 Wire Notes Line
@@
 	1    0    0    -1
 $EndComp
+Wire Wire Line
+	8950 2600 9850 2600
+Wire Wire Line
+	9800 2750 9800 2700
+Wire Wire Line
+	9800 2700 9850 2700
+Wire Wire Line
+	9300 2750 9300 2800
+Wire Wire Line
+	9300 2750 9800 2750
+Wire Wire Line
+	5150 2400 5850 2400
+Text Label 2200 6050 0    50   ~ 0
+OSC_IN
+Wire Wire Line
+	2650 6050 2100 6050
+Wire Wire Line
+	5250 1400 5250 2050
+NoConn ~ 2650 6350
+NoConn ~ 4800 2600
+Wire Wire Line
+	9850 2200 9650 2200
+Wire Wire Line
+	9850 2300 9800 2300
+Wire Wire Line
+	9800 1800 9800 2300
+Text Label 8800 1900 0    50   ~ 0
+USB_P
+Text Label 8800 1800 0    50   ~ 0
+USB_N
 $EndSCHEMATC

Commit message: hardware: sch: add some spice models to passives
Identify passives and implement the various spice models.

Signed-off-by: Sean Cross <sean@xobs.io>
Parts:
- C1, C10, C13, C16, C17, C19, C2, C24, C25, C3, C5, C8, C9: Spice_Model (none) -> 1u; Spice_Netlist_Enabled (none) -> Y; Spice_Primitive (none) -> C
- C11, C15, C20, C21, C28, C4, C7: Spice_Model (none) -> 100n; Spice_Netlist_Enabled (none) -> Y; Spice_Primitive (none) -> C
- C14, C18, C26, C27, C6: Spice_Model (none) -> 10n; Spice_Netlist_Enabled (none) -> Y; Spice_Primitive (none) -> C
- R1, R5: Spice_Model (none) -> 10k; Spice_Netlist_Enabled (none) -> Y; Spice_Primitive (none) -> R
- R11, R12: Spice_Model (none) -> 22; Spice_Netlist_Enabled (none) -> Y; Spice_Primitive (none) -> R
- R9: Spice_Model (none) -> 1.5k; Spice_Netlist_Enabled (none) -> Y; Spice_Primitive (none) -> R
- SW2: symbol tomu-fpga:PADS -> tomu-fpga-rescue:PADS-tomu-fpga
- TP1, TP10, TP11, TP12, TP2, TP3, TP4, TP5, TP6, TP7, TP8, TP9: symbol tomu-fpga:Testpoint -> tomu-fpga-rescue:Testpoint-tomu-fpga
- U1, U2, U3, U6: symbol tomu-fpga:LDO-X2SON -> tomu-fpga-rescue:LDO-X2SON-tomu-fpga
- U10: symbol tomu-fpga:RGB-LED -> tomu-fpga-rescue:RGB-LED-tomu-fpga
- U4: symbol tomu-fpga:SPI-Flash -> tomu-fpga-rescue:SPI-Flash-tomu-fpga
- U5: symbol tomu-fpga:ICE40UP5K-UWG30 -> tomu-fpga-rescue:ICE40UP5K-UWG30-tomu-fpga
- U7: symbol tomu-fpga:Oscillator -> tomu-fpga-rescue:Oscillator-tomu-fpga
- U9: symbol tomu-fpga:USB-B -> tomu-fpga-rescue:USB-B-tomu-fpga
- XX1: symbol tomu-fpga:Touchpad-Note -> tomu-fpga-rescue:Touchpad-Note-tomu-fpga; Spice_Model (none) -> Touchpad Mask Removal; Spice_Netlist_Enabled (none) -> N; Spice_Primitive (none) -> X
- XX2: symbol tomu-fpga:Case -> tomu-fpga-rescue:Case-tomu-fpga; Spice_Model (none) -> Case; Spice_Netlist_Enabled (none) -> N; Spice_Primitive (none) -> X
- XX3: symbol tomu-fpga:Case -> tomu-fpga-rescue:Case-tomu-fpga; Spice_Model (none) -> ESD Bag; Spice_Netlist_Enabled (none) -> N; Spice_Primitive (none) -> X

Commit message: hardware: sch: remove excess decoupling caps
We probably don't need 10nF, because this won't do any very-high-speed
(>100 MHz) operations.  We can think about putting them back in later,
space permitting.

Additionally, remove an extra bank of caps for one of the IO pads.
We'll double-up on capacitors there, which should be alright given the
close proximity and the fact that the only thing on that IO bank is
captouch.

Signed-off-by: Sean Cross <sean@xobs.io>
Parts:
- removed C13: 0201, 1uF, 10V, X5R, 20%, tomu-fpga:C_0201_0603Metric, symbol Device:C_Small
- removed C14, C18, C26, C27, C6: 0201, 10nF, 10V, X5R, 20%, tomu-fpga:C_0201_0603Metric, symbol Device:C_Small
- removed C15: 0201, 100nF, 10V, X5R, 20%, tomu-fpga:C_0201_0603Metric, symbol Device:C_Small
Connections:
- wire segments 236 -> 217
- no-connect marks 5 -> 3
Other:
- moved on the sheet: R1
Changed lines of the file:
@@
 L Device:R_Small R1
 U 1 1 5C0F3302
-P 2550 5000
-F 0 "R1" V 2550 5000 50  0000 C CNN
-F 1 "0201, 10k, 1/16W" H 2700 4900 50  0000 C CNN
-F 2 "tomu-fpga:R_0201_0603Metric" H 2550 5000 50  0001 C CNN
-F 3 "" H 2550 5000 50  0001 C CNN
-F 4 "ANY" H 2550 5000 50  0001 C CNN "MPN"
-F 5 "ANY" H 2550 5000 50  0001 C CNN "Manufacturer"
-F 6 "ANY" H -1000 0   50  0001 C CNN "MYPN"
-F 7 "R" H 2550 5000 50  0001 C CNN "Spice_Primitive"
-F 8 "10k" H 2550 5000 50  0001 C CNN "Spice_Model"
-F 9 "Y" H 2550 5000 50  0001 C CNN "Spice_Netlist_Enabled"
-	1    2550 5000
-	-1   0    0    1
-$EndComp
-Wire Wire Line
-	2550 4850 2550 4900
+P 2550 5150
+F 0 "R1" V 2550 5150 50  0000 C CNN
+F 1 "0201, 10k, 1/16W" H 2700 5050 50  0000 C CNN
+F 2 "tomu-fpga:R_0201_0603Metric" H 2550 5150 50  0001 C CNN
+F 3 "" H 2550 5150 50  0001 C CNN
+F 4 "ANY" H 2550 5150 50  0001 C CNN "MPN"
+F 5 "ANY" H 2550 5150 50  0001 C CNN "Manufacturer"
+F 6 "ANY" H -1000 150 50  0001 C CNN "MYPN"
+F 7 "R" H 2550 5150 50  0001 C CNN "Spice_Primitive"
+F 8 "10k" H 2550 5150 50  0001 C CNN "Spice_Model"
+F 9 "Y" H 2550 5150 50  0001 C CNN "Spice_Netlist_Enabled"
+	1    2550 5150
+	-1   0    0    1
+$EndComp
+Wire Wire Line
+	2550 4850 2550 5050
 Wire Notes Line
 	600  4250 600  7450
@@
 	8700 5200 8850 5200
 $Comp
-L Device:C_Small C18
-U 1 1 5C64A04D
-P 8450 5300
-F 0 "C18" H 8550 5300 50  0000 L CNN
-F 1 "0201, 10nF, 10V, X5R, 20%" H 7700 5200 50  0000 L CNN
-F 2 "tomu-fpga:C_0201_0603Metric" H 8450 5300 50  0001 C CNN
-F 3 "" H 8450 5300 50  0001 C CNN
-F 4 "ANY" H 200 100 50  0001 C CNN "MPN"
-F 5 "ANY" H 200 100 50  0001 C CNN "MYPN"
-F 6 "ANY" H 200 100 50  0001 C CNN "Manufacturer"
-F 7 "10n" H 0   0   50  0001 C CNN "Spice_Model"
-F 8 "Y" H 0   0   50  0001 C CNN "Spice_Netlist_Enabled"
-F 9 "C" H 0   0   50  0001 C CNN "Spice_Primitive"
-	1    8450 5300
-	1    0    0    -1
-$EndComp
-$Comp
 L Device:C_Small C17
 U 1 1 5C64A110
@@
 	8850 5300 8850 5200
 Connection ~ 8850 5200
-Wire Wire Line
-	8350 5200 8450 5200
 Connection ~ 8700 5200
 Wire Wire Line
@@
 	8600 5600 8600 5700
 Wire Wire Line
-	8450 5400 8450 5600
-Wire Wire Line
-	8450 5600 8600 5600
-Wire Wire Line
-	8450 5600 7950 5600
-Wire Wire Line
 	7950 5600 7950 5300
-Connection ~ 8450 5600
-$Comp
-L Device:C_Small C13
-U 1 1 5C71BA4C
-P 5800 950
-F 0 "C13" H 5650 1000 50  0000 L CNN
-F 1 "0201, 1uF, 10V, X5R, 20%" H 4950 900 50  0000 L CNN
-F 2 "tomu-fpga:C_0201_0603Metric" H 5800 950 50  0001 C CNN
-F 3 "" H 5800 950 50  0001 C CNN
-F 4 "ANY" H 200 -600 50  0001 C CNN "MPN"
-F 5 "ANY" H 200 -600 50  0001 C CNN "MYPN"
-F 6 "ANY" H 200 -600 50  0001 C CNN "Manufacturer"
-F 7 "C" H 5800 950 50  0001 C CNN "Spice_Primitive"
-F 8 "1u" H 5800 950 50  0001 C CNN "Spice_Model"
-F 9 "Y" H 5800 950 50  0001 C CNN "Spice_Netlist_Enabled"
-	1    5800 950
-	1    0    0    -1
-$EndComp
-$Comp
-L Device:C_Small C14
-U 1 1 5C71BAD4
-P 6150 950
-F 0 "C14" H 6000 1000 50  0000 L CNN
-F 1 "0201, 10nF, 10V, X5R, 20%" H 5400 1100 50  0000 L CNN
-F 2 "tomu-fpga:C_0201_0603Metric" H 6150 950 50  0001 C CNN
-F 3 "" H 6150 950 50  0001 C CNN
-F 4 "ANY" H 200 -600 50  0001 C CNN "MPN"
-F 5 "ANY" H 200 -600 50  0001 C CNN "MYPN"
-F 6 "ANY" H 200 -600 50  0001 C CNN "Manufacturer"
-F 7 "C" H 6150 950 50  0001 C CNN "Spice_Primitive"
-F 8 "10n" H 6150 950 50  0001 C CNN "Spice_Model"
-F 9 "Y" H 6150 950 50  0001 C CNN "Spice_Netlist_Enabled"
-	1    6150 950
-	1    0    0    -1
-$EndComp
-$Comp
-L Device:C_Small C15
-U 1 1 5C71BB44
-P 6500 950
-F 0 "C15" H 6350 1000 50  0000 L CNN
-F 1 "0201, 100nF, 10V, X5R, 20%" H 6000 750 50  0000 L CNN
-F 2 "tomu-fpga:C_0201_0603Metric" H 6500 950 50  0001 C CNN
-F 3 "" H 6500 950 50  0001 C CNN
-F 4 "ANY" H 200 -600 50  0001 C CNN "MPN"
-F 5 "ANY" H 200 -600 50  0001 C CNN "MYPN"
-F 6 "ANY" H 200 -600 50  0001 C CNN "Manufacturer"
-F 7 "C" H 6500 950 50  0001 C CNN "Spice_Primitive"
-F 8 "100n" H 6500 950 50  0001 C CNN "Spice_Model"
-F 9 "Y" H 6500 950 50  0001 C CNN "Spice_Netlist_Enabled"
-	1    6500 950
-	1    0    0    -1
-$EndComp
-Wire Wire Line
-	6750 850  6500 850
-Wire Wire Line
-	5800 850  6150 850
-Connection ~ 6150 850
-Connection ~ 6500 850
-Wire Wire Line
-	6500 850  6150 850
 Wire Wire Line
 	6750 1200 6450 1200
 Wire Wire Line
 	6750 850  6750 1200
-Wire Wire Line
-	6500 1050 6150 1050
-Connection ~ 6150 1050
-Wire Wire Line
-	6150 1050 5900 1050
-$Comp
-L power:GND #PWR026
-U 1 1 5C78A49F
-P 5900 1150
-F 0 "#PWR026" H 5900 900 50  0001 C CNN
-F 1 "GND" H 5905 977 50  0000 C CNN
-F 2 "" H 5900 1150 50  0001 C CNN
-F 3 "" H 5900 1150 50  0001 C CNN
-	1    5900 1150
-	1    0    0    -1
-$EndComp
-Wire Wire Line
-	5900 1150 5900 1050
-Connection ~ 5900 1050
-Wire Wire Line
-	5900 1050 5800 1050
-Connection ~ 6750 850
 $Comp
 L power:+3V3 #PWR040
@@
 $EndComp
 $Comp
-L Device:C_Small C26
-U 1 1 5C7EE944
-P 10250 950
-F 0 "C26" H 10100 1000 50  0000 L CNN
-F 1 "0201, 10nF, 10V, X5R, 20%" H 9500 1100 50  0000 L CNN
-F 2 "tomu-fpga:C_0201_0603Metric" H 10250 950 50  0001 C CNN
-F 3 "" H 10250 950 50  0001 C CNN
-F 4 "ANY" H 650 100 50  0001 C CNN "MPN"
-F 5 "ANY" H 650 100 50  0001 C CNN "MYPN"
-F 6 "ANY" H 650 100 50  0001 C CNN "Manufacturer"
-F 7 "10n" H 0   0   50  0001 C CNN "Spice_Model"
-F 8 "Y" H 0   0   50  0001 C CNN "Spice_Netlist_Enabled"
-F 9 "C" H 0   0   50  0001 C CNN "Spice_Primitive"
-	1    10250 950
-	1    0    0    -1
-$EndComp
-$Comp
 L Device:C_Small C28
 U 1 1 5C7EE94A
@@
 Wire Wire Line
 	10850 850  10600 850
-Wire Wire Line
-	9900 850  10250 850
-Connection ~ 10250 850
 Connection ~ 10600 850
-Wire Wire Line
-	10600 850  10250 850
 Wire Wire Line
 	10850 850  10850 1200
 Connection ~ 10850 850
-Wire Wire Line
-	10600 1050 10250 1050
-Connection ~ 10250 1050
-Wire Wire Line
-	10250 1050 10050 1050
 $Comp
 L power:GND #PWR039
@@
 $EndComp
 $Comp
-L Device:C_Small C6
-U 1 1 5C8902B0
-P 1500 4950
-F 0 "C6" H 1250 4950 50  0000 L CNN
-F 1 "0201, 10nF, 10V, X5R, 20%" H 1050 4850 50  0000 L CNN
-F 2 "tomu-fpga:C_0201_0603Metric" H 1500 4950 50  0001 C CNN
-F 3 "" H 1500 4950 50  0001 C CNN
-F 4 "ANY" H -3550 500 50  0001 C CNN "MPN"
-F 5 "ANY" H -3550 500 50  0001 C CNN "MYPN"
-F 6 "ANY" H -3550 500 50  0001 C CNN "Manufacturer"
-F 7 "10n" H 0   0   50  0001 C CNN "Spice_Model"
-F 8 "Y" H 0   0   50  0001 C CNN "Spice_Netlist_Enabled"
-F 9 "C" H 0   0   50  0001 C CNN "Spice_Primitive"
-	1    1500 4950
-	1    0    0    -1
-$EndComp
-$Comp
 L Device:C_Small C7
 U 1 1 5C8902B6
@@
 	8450 5000 7550 5000
 $Comp
-L Device:C_Small C27
-U 1 1 5BECECF0
-P 10500 5900
-F 0 "C27" H 10600 5900 50  0000 L CNN
-F 1 "0201, 10nF, 10V, X5R, 20%" H 9800 5800 50  0000 L CNN
-F 2 "tomu-fpga:C_0201_0603Metric" H 10500 5900 50  0001 C CNN
-F 3 "" H 10500 5900 50  0001 C CNN
-F 4 "ANY" H 2250 700 50  0001 C CNN "MPN"
-F 5 "ANY" H 2250 700 50  0001 C CNN "MYPN"
-F 6 "ANY" H 2250 700 50  0001 C CNN "Manufacturer"
-F 7 "10n" H 0   0   50  0001 C CNN "Spice_Model"
-F 8 "Y" H 0   0   50  0001 C CNN "Spice_Netlist_Enabled"
-F 9 "C" H 0   0   50  0001 C CNN "Spice_Primitive"
-	1    10500 5900
-	1    0    0    -1
-$EndComp
-$Comp
 L Device:C_Small C25
 U 1 1 5BECED7C
@@
 Wire Wire Line
 	9500 5550 9500 5600
-Wire Wire Line
-	10000 5650 10500 5650
-Wire Wire Line
-	10500 5650 10500 5800
-Connection ~ 10000 5650
-Wire Wire Line
-	10500 6000 10500 6100
-Wire Wire Line
-	10500 6100 10000 6100
 Connection ~ 9500 6100
 Wire Wire Line
@@
 Wire Wire Line
 	10000 5900 10000 6100
-Connection ~ 10000 6100
 Wire Wire Line
 	10000 6100 9500 6100
@@
 	600  4250 4300 4250
 Wire Wire Line
-	1500 5050 1500 5350
-Wire Wire Line
 	1900 5250 1900 5350
 Wire Wire Line
@@
 Wire Wire Line
 	1100 4650 1100 4600
-Wire Wire Line
-	1100 4600 1500 4600
 Connection ~ 1700 4600
 Wire Wire Line
-	1700 4600 1500 4600
-Wire Wire Line
 	1900 4600 1900 4850
-Wire Wire Line
-	1500 4600 1500 4850
-Connection ~ 1500 4600
 Connection ~ 2550 4850
-Connection ~ 8450 5200
-Wire Wire Line
-	8450 5200 8700 5200
 Wire Wire Line
 	1700 4600 1900 4600
@@
 $EndComp
 NoConn ~ 2650 5950
-NoConn ~ 1450 1200
 Wire Wire Line
 	8700 1800 9300 1800
@@
 	2650 6150 2550 6150
 Wire Wire Line
-	2550 5100 2550 6150
+	2550 5250 2550 6150
 Wire Wire Line
 	3400 5300 3400 4850
@@
 	5250 1400 5250 2050
 NoConn ~ 2650 6350
-NoConn ~ 4800 2600
 Wire Wire Line
 	9850 2200 9650 2200
@@
 Text Label 8800 1800 0    50   ~ 0
 USB_N
+Wire Wire Line
+	9900 850  10600 850
+Wire Wire Line
+	10050 1050 10600 1050
+Wire Wire Line
+	8350 5200 8700 5200
+Wire Wire Line
+	7950 5600 8600 5600
+Wire Wire Line
+	1100 4600 1700 4600
 $EndSCHEMATC

Commit message: hardware: sch: remove "-rescue" and "-tomu-fpga"
Somehow, KiCad added these strings to the parts libraries, which
resulted in referencing a file that didn't exist.

Remove them.

Signed-off-by: Sean Cross <sean@xobs.io>
Parts:
- SW2: symbol tomu-fpga-rescue:PADS-tomu-fpga -> tomu-fpga:PADS
- TP1, TP10, TP11, TP12, TP2, TP3, TP4, TP5, TP6, TP7, TP8, TP9: symbol tomu-fpga-rescue:Testpoint-tomu-fpga -> tomu-fpga:Testpoint
- U1, U2, U3, U6: symbol tomu-fpga-rescue:LDO-X2SON-tomu-fpga -> tomu-fpga:LDO-X2SON
- U10: symbol tomu-fpga-rescue:RGB-LED-tomu-fpga -> tomu-fpga:RGB-LED
- U4: symbol tomu-fpga-rescue:SPI-Flash-tomu-fpga -> tomu-fpga:SPI-Flash
- U5: symbol tomu-fpga-rescue:ICE40UP5K-UWG30-tomu-fpga -> tomu-fpga:ICE40UP5K-UWG30
- U7: symbol tomu-fpga-rescue:Oscillator-tomu-fpga -> tomu-fpga:Oscillator
- U9: symbol tomu-fpga-rescue:USB-B-tomu-fpga -> tomu-fpga:USB-B
- XX1: symbol tomu-fpga-rescue:Touchpad-Note-tomu-fpga -> tomu-fpga:Touchpad-Note
- XX2, XX3: symbol tomu-fpga-rescue:Case-tomu-fpga -> tomu-fpga:Case
Changed lines of the file:
@@
 Connection ~ 1150 2100
 $Comp
-L tomu-fpga-rescue:USB-B-tomu-fpga U9
+L tomu-fpga:USB-B U9
 U 1 1 5BD8B24F
 P 8300 1600
@@
 $EndComp
 $Comp
-L tomu-fpga-rescue:RGB-LED-tomu-fpga U10
+L tomu-fpga:RGB-LED U10
 U 1 1 5BD90F18
 P 8550 2850
@@
 $EndComp
 $Comp
-L tomu-fpga-rescue:PADS-tomu-fpga SW2
+L tomu-fpga:PADS SW2
 U 1 1 5BE44C19
 P 5300 1200
@@
 	10000 6100 9500 6100
 $Comp
-L tomu-fpga-rescue:Oscillator-tomu-fpga U7
+L tomu-fpga:Oscillator U7
 U 1 1 5C0E8D0F
 P 4800 2350
@@
 CDONE
 $Comp
-L tomu-fpga-rescue:ICE40UP5K-UWG30-tomu-fpga U5
+L tomu-fpga:ICE40UP5K-UWG30 U5
 U 3 1 5C122A3A
 P 6450 1750
@@
 $EndComp
 $Comp
-L tomu-fpga-rescue:ICE40UP5K-UWG30-tomu-fpga U5
+L tomu-fpga:ICE40UP5K-UWG30 U5
 U 4 1 5C122B60
 P 10200 4800
@@
 $EndComp
 $Comp
-L tomu-fpga-rescue:SPI-Flash-tomu-fpga U4
+L tomu-fpga:SPI-Flash U4
 U 1 1 5C1645BF
 P 1650 7000
@@
 	4950 2150 5850 2150
 $Comp
-L tomu-fpga-rescue:ICE40UP5K-UWG30-tomu-fpga U5
+L tomu-fpga:ICE40UP5K-UWG30 U5
 U 1 1 5C1225F9
 P 10400 2400
@@
 	9000 5000 9600 5000
 $Comp
-L tomu-fpga-rescue:LDO-X2SON-tomu-fpga U1
+L tomu-fpga:LDO-X2SON U1
 U 1 1 5BF1A34B
 P 1650 1300
@@
 	2050 1150 2050 1250
 $Comp
-L tomu-fpga-rescue:LDO-X2SON-tomu-fpga U2
+L tomu-fpga:LDO-X2SON U2
 U 1 1 5BF61C95
 P 1650 2400
@@
 	1300 1800 1300 2350
 $Comp
-L tomu-fpga-rescue:LDO-X2SON-tomu-fpga U3
+L tomu-fpga:LDO-X2SON U3
 U 1 1 5BFAB7F1
 P 1650 3500
@@
 	2050 3450 2050 3600
 $Comp
-L tomu-fpga-rescue:LDO-X2SON-tomu-fpga U6
+L tomu-fpga:LDO-X2SON U6
 U 1 1 5BFF652A
 P 8150 4800
@@
 	7850 4500 7850 4750
 $Comp
-L tomu-fpga-rescue:Testpoint-tomu-fpga TP2
+L tomu-fpga:Testpoint TP2
 U 1 1 5C03018F
 P 5250 4500
@@
 SPI_MISO
 $Comp
-L tomu-fpga-rescue:Testpoint-tomu-fpga TP3
+L tomu-fpga:Testpoint TP3
 U 1 1 5C042DE8
 P 5250 4650
@@
 	5400 4700 5850 4700
 $Comp
-L tomu-fpga-rescue:Testpoint-tomu-fpga TP4
+L tomu-fpga:Testpoint TP4
 U 1 1 5C068EF3
 P 5250 4800
@@
 	5400 4850 5850 4850
 $Comp
-L tomu-fpga-rescue:Testpoint-tomu-fpga TP5
+L tomu-fpga:Testpoint TP5
 U 1 1 5C068EFC
 P 5250 4950
@@
 SPI_IO3
 $Comp
-L tomu-fpga-rescue:Testpoint-tomu-fpga TP6
+L tomu-fpga:Testpoint TP6
 U 1 1 5C07C50C
 P 5250 5100
@@
 $EndComp
 $Comp
-L tomu-fpga-rescue:Testpoint-tomu-fpga TP7
+L tomu-fpga:Testpoint TP7
 U 1 1 5C07C63D
 P 5250 5250
@@
 CRESET
 $Comp
-L tomu-fpga-rescue:Testpoint-tomu-fpga TP8
+L tomu-fpga:Testpoint TP8
 U 1 1 5C0A39C6
 P 5250 5400
@@
 CDONE
 $Comp
-L tomu-fpga-rescue:Testpoint-tomu-fpga TP9
+L tomu-fpga:Testpoint TP9
 U 1 1 5C0B4DBE
 P 5250 5550
@@
 	5400 5600 5850 5600
 $Comp
-L tomu-fpga-rescue:Testpoint-tomu-fpga TP1
+L tomu-fpga:Testpoint TP1
 U 1 1 5C0C6529
 P 5250 4350
@@
 $EndComp
 $Comp
-L tomu-fpga-rescue:Testpoint-tomu-fpga TP12
+L tomu-fpga:Testpoint TP12
 U 1 1 5C0C65AF
 P 5250 6000
@@
 USB_N
 $Comp
-L tomu-fpga-rescue:Testpoint-tomu-fpga TP10
+L tomu-fpga:Testpoint TP10
 U 1 1 5C0EA6CF
 P 5250 5700
@@
 $EndComp
 $Comp
-L tomu-fpga-rescue:Testpoint-tomu-fpga TP11
+L tomu-fpga:Testpoint TP11
 U 1 1 5C0EA757
 P 5250 5850
@@
 	3850 7250 3850 6900
 $Comp
-L tomu-fpga-rescue:ICE40UP5K-UWG30-tomu-fpga U5
+L tomu-fpga:ICE40UP5K-UWG30 U5
 U 2 1 5C122971
 P 3250 6500
@@
 Test Pads
 $Comp
-L tomu-fpga-rescue:Touchpad-Note-tomu-fpga XX1
+L tomu-fpga:Touchpad-Note XX1
 U 1 1 5C0024CC
 P 5900 3500
@@
 $EndComp
 $Comp
-L tomu-fpga-rescue:Case-tomu-fpga XX2
+L tomu-fpga:Case XX2
 U 1 1 5C011D36
 P 5900 3750
@@
 Manufacturing Notes
 $Comp
-L tomu-fpga-rescue:Case-tomu-fpga XX3
+L tomu-fpga:Case XX3
 U 1 1 5C0476E4
 P 5250 3450

Commit message: hardware: sch: add esd diodes
These will be placed on the USB lines as well as the captouch lines.

Signed-off-by: Sean Cross <sean@xobs.io>
Parts:
- added D1, D2, D3, D4, D5, D6, D7: D5V0L1B2LP3-7, tomu-fpga:X1-DFN1006-2, symbol Device:D_Small
Connections:
- wire segments 217 -> 250
Other:
- note added: "Captouch Input"
- note removed: "Oscillator and Captouch"
- moved on the sheet: C11, C24, C28, C5, C7, U7

Commit message: hardware: sch: define spi part numbers for dvt board
This part is smaller.  Define both the part number and an alternative
part number.

Signed-off-by: Sean Cross <sean@xobs.io>
Parts:
- U4: AManufacturer (none) -> Macronix; APN (none) -> MX25R1635FZUIH0; DPN W25Q128JVSIMCT-ND -> 1970-1011-6-ND; MPN W25Q128JVSIM -> GD25Q16CEIGR; Manufacturer Winbond Electronics -> GigaDevice Semiconductor (HK) Limited
Connections:
- wire segments 250 -> 255
Other:
- moved on the sheet: C17, C19, C24, C28
