File: hardware/pcb/tomu-fpga.sch (KiCad schematic (older format))
At the start: 55 parts, among them SW2 Captouch Pads, U1 LDO-X2SON-1.2V, U10 RGB-LED, U2 LDO-X2SON-3.3V, U3 LDO-X2SON-2.5V, U4 SPI Flash, U5 ICE40UP5K-UWG30, U6 LDO-X2SON-1.2V, U7 Crystal Oscillator, U9 USB-B

Commit message: hardware: sch: add column for "DNP"
After discussing with one factory, this is their preferred method of
indicating a part is "Do-Not-Populate".

Signed-off-by: Sean Cross <sean@xobs.io>
Parts:
- SW2, TP1, TP10, TP11, TP12, TP2, TP3, TP4, TP5, TP6, TP7, TP8, TP9, U9, XX1, XX2, XX3: DNP (none) -> X
- U4: AManufacturer Macronix -> Macronix
Changed lines of the file:
@@
 F 6 "DNP" H 8300 1600 50  0001 C CNN "MYPN"
 F 7 "PCB-etched USB pads" H 0   0   50  0001 C CNN "Description"
+F 8 "X" H 0   0   50  0001 C CNN "DNP"
 	1    8300 1600
 	-1   0    0    1
@@
 F 6 "DNP" H 5300 1200 50  0001 C CNN "MYPN"
 F 7 "PCB-etched captouch pads" H -200 -1000 50  0001 C CNN "Description"
+F 8 "X" V 5300 1200 50  0001 C CNN "DNP"
 	1    5300 1200
 	0    -1   -1   0
@@
 F 7 "IC FLASH 128M SPI 133MHZ 8SOIC" H 0   0   50  0001 C CNN "Description"
 F 8 "MX25R1635FZUIH0" H 1650 7000 50  0001 C CNN "APN"
-F 9 " Macronix" H 1650 7000 50  0001 C CNN "AManufacturer"
+F 9 "Macronix" H 1650 7000 50  0001 C CNN "AManufacturer"
 	1    1650 7000
 	1    0    0    -1
@@
 F 2 "tomu-fpga:testpoint" H 5250 4500 50  0001 C CNN
 F 3 "" H 5250 4500 50  0001 C CNN
+F 4 "X" H 0   0   50  0001 C CNN "DNP"
 	1    5250 4500
 	-1   0    0    1
@@
 F 2 "tomu-fpga:testpoint" H 5250 4650 50  0001 C CNN
 F 3 "" H 5250 4650 50  0001 C CNN
+F 4 "X" H 0   0   50  0001 C CNN "DNP"
 	1    5250 4650
 	-1   0    0    1
@@
 F 2 "tomu-fpga:testpoint" H 5250 4800 50  0001 C CNN
 F 3 "" H 5250 4800 50  0001 C CNN
+F 4 "X" H 0   0   50  0001 C CNN "DNP"
 	1    5250 4800
 	-1   0    0    1
@@
 F 2 "tomu-fpga:testpoint" H 5250 4950 50  0001 C CNN
 F 3 "" H 5250 4950 50  0001 C CNN
+F 4 "X" H 0   0   50  0001 C CNN "DNP"
 	1    5250 4950
 	-1   0    0    1
@@
 F 2 "tomu-fpga:testpoint" H 5250 5100 50  0001 C CNN
 F 3 "" H 5250 5100 50  0001 C CNN
+F 4 "X" H 0   0   50  0001 C CNN "DNP"
 	1    5250 5100
 	-1   0    0    1
@@
 F 2 "tomu-fpga:testpoint" H 5250 5250 50  0001 C CNN
 F 3 "" H 5250 5250 50  0001 C CNN
+F 4 "X" H 0   0   50  0001 C CNN "DNP"
 	1    5250 5250
 	-1   0    0    1
@@
 F 2 "tomu-fpga:testpoint" H 5250 5400 50  0001 C CNN
 F 3 "" H 5250 5400 50  0001 C CNN
+F 4 "X" H 0   0   50  0001 C CNN "DNP"
 	1    5250 5400
 	-1   0    0    1
@@
 F 2 "tomu-fpga:testpoint" H 5250 5550 50  0001 C CNN
 F 3 "" H 5250 5550 50  0001 C CNN
+F 4 "X" H 0   0   50  0001 C CNN "DNP"
 	1    5250 5550
 	-1   0    0    1
@@
 F 2 "tomu-fpga:testpoint" H 5250 4350 50  0001 C CNN
 F 3 "" H 5250 4350 50  0001 C CNN
+F 4 "X" H 0   0   50  0001 C CNN "DNP"
 	1    5250 4350
 	-1   0    0    1
@@
 F 2 "tomu-fpga:testpoint" H 5250 6000 50  0001 C CNN
 F 3 "" H 5250 6000 50  0001 C CNN
+F 4 "X" H 0   0   50  0001 C CNN "DNP"
 	1    5250 6000
 	-1   0    0    1
@@
 F 2 "tomu-fpga:testpoint" H 5250 5700 50  0001 C CNN
 F 3 "" H 5250 5700 50  0001 C CNN
+F 4 "X" H 0   0   50  0001 C CNN "DNP"
 	1    5250 5700
 	-1   0    0    1
@@
 F 2 "tomu-fpga:testpoint" H 5250 5850 50  0001 C CNN
 F 3 "" H 5250 5850 50  0001 C CNN
+F 4 "X" H 0   0   50  0001 C CNN "DNP"
 	1    5250 5850
 	-1   0    0    1
@@
 F 8 "Touchpad Mask Removal" H 5900 3500 50  0001 C CNN "Spice_Model"
 F 9 "N" H 5900 3500 50  0001 C CNN "Spice_Netlist_Enabled"
+F 10 "X" H 0   0   50  0001 C CNN "DNP"
 	1    5900 3500
 	1    0    0    -1
@@
 F 8 "Case" H 5900 3750 50  0001 C CNN "Spice_Model"
 F 9 "N" H 5900 3750 50  0001 C CNN "Spice_Netlist_Enabled"
+F 10 "X" H 0   0   50  0001 C CNN "DNP"
 	1    5900 3750
 	1    0    0    -1
@@
 F 8 "ESD Bag" H 5250 3450 50  0001 C CNN "Spice_Model"
 F 9 "N" H 5250 3450 50  0001 C CNN "Spice_Netlist_Enabled"
+F 10 "X" H 0   0   50  0001 C CNN "DNP"
 	1    5250 3450
 	1    0    0    -1
